File: kicad/weather/weather.kicad_pcb (KiCad board)
At the start: 2 copper layers, 61.5 x 34 mm, 7 parts

Commit message: Documentation & KiCad update
Routing:
- net /DIS_RST: track 37.6 -> 54.1 mm
- net BAT: track 50.8 -> 49.6 mm, vias 0 -> 1
- net 3V3: track 46.0 -> 46.2 mm, vias 1 -> 0
